Commit message: fix: restructure ros2_control xacro, add sim_time param, reduce reference_timeout

File: description/prius_gazebo.xacro (robot description, xacro)
@@ -4,4 +4,5 @@
     <plugin name="gazebo_ros2_control" filename="libgazebo_ros2_control.so">
       <parameters>$(find gcamp_gazebo)/config/prius_controllers.yaml</parameters>
+      <parameters>$(find gcamp_gazebo)/config/gaz_ros2_ctl_use_sim.yaml</parameters>
     </plugin>
   </gazebo>

File: description/prius_ros2_control.xacro (robot description, xacro)
@@ -1,58 +1,101 @@
 <?xml version="1.0"?>
 <robot xmlns:xacro="http://www.ros.org/wiki/xacro">
-  <xacro:arg name="use_ros2_control" default="true"/>
-  <xacro:arg name="sim_mode"         default="false"/>
   <xacro:if value="$(arg use_ros2_control)">
-    <ros2_control name="GazeboSystem" type="system">
-      <hardware>
-        <xacro:if value="$(arg sim_mode)">
+    <xacro:if value="$(arg sim_mode)">
+      <ros2_control name="GazeboSystem" type="system">
+        <hardware>
           <plugin>gazebo_ros2_control/GazeboSystem</plugin>
-        </xacro:if>
-        <xacro:unless value="$(arg sim_mode)">
+        </hardware>
+        <joint name="front_left_steering_joint">
+          <command_interface name="position">
+            <param name="min">-0.5</param>
+            <param name="max">0.5</param>
+          </command_interface>
+          <state_interface name="position"/>
+          <state_interface name="velocity"/>
+        </joint>
+        <joint name="front_right_steering_joint">
+          <command_interface name="position">
+            <param name="min">-0.5</param>
+            <param name="max">0.5</param>
+          </command_interface>
+          <state_interface name="position"/>
+          <state_interface name="velocity"/>
+        </joint>
+        <joint name="rear_left_wheel_joint">
+          <command_interface name="velocity">
+            <param name="min">-30</param>
+            <param name="max">30</param>
+          </command_interface>
+          <state_interface name="velocity"/>
+          <state_interface name="position"/>
+        </joint>
+        <joint name="rear_right_wheel_joint">
+          <command_interface name="velocity">
+            <param name="min">-30</param>
+            <param name="max">30</param>
+          </command_interface>
+          <state_interface name="velocity"/>
+          <state_interface name="position"/>
+        </joint>
+        <!-- Front wheel joints: state only (free spinning, no drive command) -->
+        <joint name="front_left_wheel_joint">
+          <state_interface name="velocity"/>
+          <state_interface name="position"/>
+        </joint>
+        <joint name="front_right_wheel_joint">
+          <state_interface name="velocity"/>
+          <state_interface name="position"/>
+        </joint>
+      </ros2_control>
+    </xacro:if>
+    <xacro:unless value="$(arg sim_mode)">
+      <ros2_control name="RealRobot" type="system">
+        <hardware>
           <plugin>mock_components/GenericSystem</plugin>
-        </xacro:unless>
-      </hardware>
-      <joint name="front_left_steering_joint">
-        <command_interface name="position">
-          <param name="min">-0.5</param>
-          <param name="max">0.5</param>
-        </command_interface>
-        <state_interface name="position"/>
-        <state_interface name="velocity"/>
-      </joint>
-      <joint name="front_right_steering_joint">
-        <command_interface name="position">
-          <param name="min">-0.5</param>
-          <param name="max">0.5</param>
-        </command_interface>
-        <state_interface name="position"/>
-        <state_interface name="velocity"/>
-      </joint>
-      <joint name="rear_left_wheel_joint">
-        <command_interface name="velocity">
-          <param name="min">-30</param>
-          <param name="max">30</param>
-        </command_interface>
-        <state_interface name="velocity"/>
-        <state_interface name="position"/>
-      </joint>
-      <joint name="rear_right_wheel_joint">
-        <command_interface name="velocity">
-          <param name="min">-30</param>
-          <param name="max">30</param>
-        </command_interface>
-        <state_interface name="velocity"/>
-        <state_interface name="position"/>
-      </joint>
-      <!-- Front wheel joints: state only (free spinning, no drive command) -->
-      <joint name="front_left_wheel_joint">
-        <state_interface name="velocity"/>
-        <state_interface name="position"/>
-      </joint>
-      <joint name="front_right_wheel_joint">
-        <state_interface name="velocity"/>
-        <state_interface name="position"/>
-      </joint>
-    </ros2_control>
+        </hardware>
+        <joint name="front_left_steering_joint">
+          <command_interface name="position">
+            <param name="min">-0.5</param>
+            <param name="max">0.5</param>
+          </command_interface>
+          <state_interface name="position"/>
+          <state_interface name="velocity"/>
+        </joint>
+        <joint name="front_right_steering_joint">
+          <command_interface name="position">
+            <param name="min">-0.5</param>
+            <param name="max">0.5</param>
+          </command_interface>
+          <state_interface name="position"/>
+          <state_interface name="velocity"/>
+        </joint>
+        <joint name="rear_left_wheel_joint">
+          <command_interface name="velocity">
+            <param name="min">-30</param>
+            <param name="max">30</param>
+          </command_interface>
+          <state_interface name="velocity"/>
+          <state_interface name="position"/>
+        </joint>
+        <joint name="rear_right_wheel_joint">
+          <command_interface name="velocity">
+            <param name="min">-30</param>
+            <param name="max">30</param>
+          </command_interface>
+          <state_interface name="velocity"/>
+          <state_interface name="position"/>
+        </joint>
+        <!-- Front wheel joints: state only (free spinning, no drive command) -->
+        <joint name="front_left_wheel_joint">
+          <state_interface name="velocity"/>
+          <state_interface name="position"/>
+        </joint>
+        <joint name="front_right_wheel_joint">
+          <state_interface name="velocity"/>
+          <state_interface name="position"/>
+        </joint>
+      </ros2_control>
+    </xacro:unless>
   </xacro:if>
 </robot>
