Commit message: fix: correct wheel inertia tensor and base_footprint convention in prius_core.xacro

File: description/prius_core.xacro (robot description, xacro)
@@ -9,11 +9,11 @@
   <xacro:property name="axle_z"       value="${wheel_radius}"/>
   <xacro:property name="max_steer"    value="0.5"/>
-  <link name="base_footprint"/>
+  <link name="base_link"/>
   <joint name="base_footprint_joint" type="fixed">
-    <parent link="base_footprint"/>
-    <child  link="base_link"/>
+    <parent link="base_link"/>
+    <child  link="base_footprint"/>
     <origin xyz="0 0 0" rpy="0 0 0"/>
   </joint>
-  <link name="base_link"/>
+  <link name="base_footprint"/>
   <joint name="chassis_joint" type="fixed">
     <parent link="base_link"/>
@@ -71,5 +71,5 @@
     <inertial>
       <mass value="11.0"/>
-      <inertia ixx="0.1" ixy="0" ixz="0" iyy="0.1" iyz="0" izz="0.1"/>
+      <inertia ixx="0.311" ixy="0" ixz="0" iyy="0.538" iyz="0" izz="0.311"/>
     </inertial>
   </link>
@@ -106,5 +106,5 @@
     <inertial>
       <mass value="11.0"/>
-      <inertia ixx="0.1" ixy="0" ixz="0" iyy="0.1" iyz="0" izz="0.1"/>
+      <inertia ixx="0.311" ixy="0" ixz="0" iyy="0.538" iyz="0" izz="0.311"/>
     </inertial>
   </link>
@@ -128,5 +128,5 @@
     <inertial>
       <mass value="11.0"/>
-      <inertia ixx="0.1" ixy="0" ixz="0" iyy="0.1" iyz="0" izz="0.1"/>
+      <inertia ixx="0.311" ixy="0" ixz="0" iyy="0.538" iyz="0" izz="0.311"/>
     </inertial>
   </link>
@@ -150,5 +150,5 @@
     <inertial>
       <mass value="11.0"/>
-      <inertia ixx="0.1" ixy="0" ixz="0" iyy="0.1" iyz="0" izz="0.1"/>
+      <inertia ixx="0.311" ixy="0" ixz="0" iyy="0.538" iyz="0" izz="0.311"/>
     </inertial>
   </link>

Commit message: fix: add 1mm sphere visuals to empty wheel and optical-frame links to prevent Ogre AABB assertion

File: description/prius_core.xacro (robot description, xacro)
@@ -22,9 +22,9 @@
   </joint>
   <link name="chassis">
-    <!-- SDF chassis pose (0,-0.266,0.48) → URDF (0.266,0,0.48); mesh rotated +90° Z -->
+    <!-- Original Prius SDF mesh has no visual pose; rotate only to map SDF Y-forward to ROS X-forward. -->
     <visual>
-      <origin xyz="0.266 0 0.48" rpy="0 0 1.5708"/>
+      <origin xyz="0 0 0" rpy="0 0 1.5708"/>
       <geometry>
-        <mesh filename="package://gcamp_gazebo/meshes/Hybrid.obj" scale="0.01 0.01 0.01"/>
+        <mesh filename="file://$(find gcamp_gazebo)/meshes/Hybrid.obj" scale="0.01 0.01 0.01"/>
       </geometry>
     </visual>
@@ -61,7 +61,5 @@
   <link name="front_left_wheel">
     <visual>
-      <origin xyz="0 0 0" rpy="${pi/2} 0 0"/>
-      <geometry><cylinder radius="${wheel_radius}" length="${wheel_width}"/></geometry>
-      <material name="dark_grey"><color rgba="0.2 0.2 0.2 1"/></material>
+      <geometry><sphere radius="0.001"/></geometry>
     </visual>
     <collision>
@@ -96,7 +94,5 @@
   <link name="front_right_wheel">
     <visual>
-      <origin xyz="0 0 0" rpy="${pi/2} 0 0"/>
-      <geometry><cylinder radius="${wheel_radius}" length="${wheel_width}"/></geometry>
-      <material name="dark_grey"/>
+      <geometry><sphere radius="0.001"/></geometry>
     </visual>
     <collision>
@@ -118,7 +114,5 @@
   <link name="rear_left_wheel">
     <visual>
-      <origin xyz="0 0 0" rpy="${pi/2} 0 0"/>
-      <geometry><cylinder radius="${wheel_radius}" length="${wheel_width}"/></geometry>
-      <material name="dark_grey"/>
+      <geometry><sphere radius="0.001"/></geometry>
     </visual>
     <collision>
@@ -140,7 +134,5 @@
   <link name="rear_right_wheel">
     <visual>
-      <origin xyz="0 0 0" rpy="${pi/2} 0 0"/>
-      <geometry><cylinder radius="${wheel_radius}" length="${wheel_width}"/></geometry>
-      <material name="dark_grey"/>
+      <geometry><sphere radius="0.001"/></geometry>
     </visual>
     <collision>

File: description/prius_sensors.xacro (robot description, xacro)
@@ -28,5 +28,9 @@
     <origin xyz="0 0 0" rpy="${-pi/2} 0 ${-pi/2}"/>
   </joint>
-  <link name="front_camera_link_optical"/>
+  <link name="front_camera_link_optical">
+    <visual>
+      <geometry><sphere radius="0.001"/></geometry>
+    </visual>
+  </link>
   <gazebo reference="front_camera_link">
     <sensor name="front_camera" type="camera">
@@ -87,5 +91,9 @@
     <origin xyz="0 0 0" rpy="${-pi/2} 0 ${-pi/2}"/>
   </joint>
-  <link name="depth_camera_link_optical"/>
+  <link name="depth_camera_link_optical">
+    <visual>
+      <geometry><sphere radius="0.001"/></geometry>
+    </visual>
+  </link>
   <gazebo reference="depth_camera_link">
     <sensor name="depth_camera" type="depth">

Commit message: fix: add sphere visuals to steer links to prevent Ogre AABB assertion

File: description/prius_core.xacro (robot description, xacro)
@@ -48,4 +48,7 @@
   </joint>
   <link name="front_left_steer_link">
+    <visual>
+      <geometry><sphere radius="0.001"/></geometry>
+    </visual>
     <inertial>
       <mass value="0.1"/>
@@ -81,4 +84,7 @@
   </joint>
   <link name="front_right_steer_link">
+    <visual>
+      <geometry><sphere radius="0.001"/></geometry>
+    </visual>
     <inertial>
       <mass value="0.1"/>
