Commit message: Integrate MobilePixor 3D LiDAR object detection pipeline
- Added detect.py, preprocess.py, and postprocess.py for real-time PyTorch inference on /points_raw
- Added JRDB-trained base_demo.json configuration
- Fixed Softmax and NMS bugs in postprocess.py to prevent false positives and clone boxes
- Implemented size filtering, dynamic TF frames, and remote toggle functionality (/enable_detection)
- Updated CMakeLists.txt to install the new AI launch files
- Modified vlp_16.xacro and small_city_sdc_prius.world to configure the simulated Velodyne LiDAR and spawn human test subjects for validation

File: description/vlp_16.xacro (robot description, xacro)
@@ -4,5 +4,5 @@
   <!-- <xacro:macro name="VLP-16" params="*origin parent:=base_link name:=velodyne topic:=/velodyne_points hz:=10 lasers:=16 samples:=1875 collision_range:=0.3 min_range:=0.9 max_range:=130.0 noise:=0.008 min_angle:=-${M_PI} max_angle:=${M_PI} vehicle_name:=vehicle"> -->
     <joint name="velodyne_joint" type="fixed">
-        <origin rpy="0 0 0" xyz="0 0 1"/>
+        <origin rpy="0 0 0" xyz="0 0.25 1.58"/>
         <parent link="base_link"/>
         <child link="velodyne"/>
@@ -84,10 +84,10 @@
             </noise>
           </ray>
-          <plugin filename="libgazebo_ros_velodyne_laser.so" name="gazebo_ros_laser_controller">
-            <topicName>/points_raw</topicName>
-            <frameName>velodyne</frameName>
-            <min_range>0.9</min_range>
-            <max_range>130.0</max_range>
-            <gaussianNoise>0.008</gaussianNoise>
+          <plugin filename="libgazebo_ros_ray_sensor.so" name="gazebo_ros_laser_controller">
+            <ros>
+              <remapping>~/out:=/points_raw</remapping>
+            </ros>
+            <output_type>sensor_msgs/PointCloud2</output_type>
+            <frame_name>velodyne</frame_name>
           </plugin>
         </sensor>
