Commit message: feat: update autonomous navigation simulation

File: description/vlp_16.xacro (robot description, xacro)
@@ -4,5 +4,5 @@
   <!-- <xacro:macro name="VLP-16" params="*origin parent:=base_link name:=velodyne topic:=/velodyne_points hz:=10 lasers:=16 samples:=1875 collision_range:=0.3 min_range:=0.9 max_range:=130.0 noise:=0.008 min_angle:=-${M_PI} max_angle:=${M_PI} vehicle_name:=vehicle"> -->
     <joint name="velodyne_joint" type="fixed">
-        <origin rpy="0 0 0" xyz="0 0.25 1.58"/>
+        <origin rpy="0 0 0" xyz="0 -0.15 2.0"/>
         <parent link="base_link"/>
         <child link="velodyne"/>
@@ -61,5 +61,5 @@
             <scan>
               <horizontal>
-                <samples>1875</samples>
+                <samples>3600</samples>
                 <resolution>1</resolution>
                 <min_angle>-3.1415926535897931</min_angle>
@@ -67,8 +67,8 @@
               </horizontal>
               <vertical>
-                <samples>16</samples>
+                <samples>64</samples>
                 <resolution>1</resolution>
-                <min_angle>-0.2617993877991494</min_angle>
-                <max_angle>0.2617993877991494</max_angle>
+                <min_angle>-0.4363323129985824</min_angle>
+                <max_angle>0.0349065850398866</max_angle>
               </vertical>
             </scan>
